Commit message: Created core URDF

File: description/robot_core.xacro (robot description, xacro)
@@ -43,4 +43,10 @@
         <material name="blue"/>
     </visual>
+    <collision>
+        <geometry>
+            <cylinder length="0.04" radius="0.05" />
+        </geometry>
+        <material name="blue"/>
+    </collision>
     <xacro:inertial_cylinder mass="0.1" length="0.05" radius="0.05">
         <origin xyz="0 0 0" rpy="0 0 0"/>
@@ -61,4 +67,10 @@
         <material name="blue"/>
     </visual>
+    <collision>
+        <geometry>
+            <cylinder length="0.04" radius="0.05" />
+        </geometry>
+        <material name="blue"/>
+    </collision>
     <xacro:inertial_sphere mass="0.1" radius="0.05">
         <origin xyz="0 0 0" rpy="0 0 0"/>
@@ -78,4 +90,10 @@
         <material name="black"/>
     </visual>
+    <collision>
+        <geometry>
+            <sphere radius="0.05" />
+        </geometry>
+        <material name="black"/>
+    </collision>
 </link>
 	<material name="white">
